File: Kicad/garden-water-system.kicad_pcb (KiCad board)
At the start: 2 copper layers, 75 x 60 mm, 35 parts, among them J1 Conn_01x02, J10 Screw_Terminal_01x05, J11 Conn_01x04, J12 Conn_01x05, J13 Jack-DC, J2 Conn_01x05, J3 Conn_01x03, J4 Conn_01x03, J5 Conn_01x03, J6 Conn_01x03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

Commit message: Add protection diode on hardware power supply
Parts:
- added D5: D, Diode_SMD:D_2010_5025Metric_Pad1.52x2.65mm_HandSolder, F.Cu at (170.5, 37.2)
Connections:
- J10 pad 1: Net-(C4-Pad1) -> Net-(D5-Pad1)
- J10 pad 2: Net-(C4-Pad1) -> Net-(D5-Pad1)
- J10 pad 3: Net-(C4-Pad1) -> Net-(D5-Pad1)
- J10 pad 4: Net-(C4-Pad1) -> Net-(D5-Pad1)
- J10 pad 5: Net-(C4-Pad1) -> Net-(D5-Pad1)
Routing:
- net Net-(C4-Pad1): track 69.7 -> 23.1 mm
- net Net-(D5-Pad1): track 0.00 -> 42.5 mm
Changed lines of the file:
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@@
     (thickness 1.6)
     (drawings 12)
-    (tracks 201)
+    (tracks 202)
     (zones 0)
-    (modules 35)
-    (nets 28)
+    (modules 36)
+    (nets 29)
   )
   (page A4)
@@
   (net 26 /clock_interrupt)
   (net 27 "Net-(R1-Pad2)")
+  (net 28 "Net-(D5-Pad1)")
   (net_class Default "This is the default net class."
     (clearance 0.2)
@@
     (uvia_drill 0.1)
     (add_net "Net-(C4-Pad1)")
+    (add_net "Net-(D5-Pad1)")
   )
   (net_class VCC ""
@@
     (uvia_drill 0.1)
     (add_net VCC)
+  )
+  (module Diode_SMD:D_2010_5025Metric_Pad1.52x2.65mm_HandSolder (layer F.Cu)
+    (at 170.5 37.25)
+    (descr "Diode SMD 2010 (5025 Metric), square (rectangular) end terminal, IPC_7351 nominal, (Body size source: http://www.tortai-tech.com/upload/download/2011102023233369053.pdf), generated with kicad-footprint-generator")
+    (tags "diode handsolder")
+    (attr smd)
+    (fp_text reference D5 (at 4.5 -1.5) (layer F.SilkS) hide
+      (effects (font (size 1 1) (thickness 0.15)))
+    )
+    (fp_text value D (at 0 2.28) (layer F.Fab)
+      (effects (font (size 1 1) (thickness 0.15)))
+    )
+    (fp_text user %R (at 0 0) (layer F.Fab)
+      (effects (font (size 1 1) (thickness 0.15)))
+    )
+    (fp_line (start 3.35 1.58) (end -3.35 1.58) (layer F.CrtYd) (width 0.05))
+    (fp_line (start 3.35 -1.58) (end 3.35 1.58) (layer F.CrtYd) (width 0.05))
+    (fp_line (start -3.35 -1.58) (end 3.35 -1.58) (layer F.CrtYd) (width 0.05))
+    (fp_line (start -3.35 1.58) (end -3.35 -1.58) (layer F.CrtYd) (width 0.05))
+    (fp_line (start -3.36 1.585) (end 2.5 1.585) (layer F.SilkS) (width 0.12))
+    (fp_line (start -3.36 -1.585) (end -3.36 1.585) (layer F.SilkS) (width 0.12))
+    (fp_line (start 2.5 -1.585) (end -3.36 -1.585) (layer F.SilkS) (width 0.12))
+    (fp_line (start 2.5 1.25) (end 2.5 -1.25) (layer F.Fab) (width 0.1))
+    (fp_line (start -2.5 1.25) (end 2.5 1.25) (layer F.Fab) (width 0.1))
+    (fp_line (start -2.5 -0.625) (end -2.5 1.25) (layer F.Fab) (width 0.1))
+    (fp_line (start -1.875 -1.25) (end -2.5 -0.625) (layer F.Fab) (width 0.1))
+    (fp_line (start 2.5 -1.25) (end -1.875 -1.25) (layer F.Fab) (width 0.1))
+    (pad 2 smd roundrect (at 2.3375 0) (size 1.525 2.65) (layers F.Cu F.Paste F.Mask) (roundrect_rratio 0.163934)
+      (net 5 "Net-(C4-Pad1)"))
+    (pad 1 smd roundrect (at -2.3375 0) (size 1.525 2.65) (layers F.Cu F.Paste F.Mask) (roundrect_rratio 0.163934)
+      (net 28 "Net-(D5-Pad1)"))
+    (model ${KISYS3DMOD}/Diode_SMD.3dshapes/D_2010_5025Metric.wrl
+      (at (xyz 0 0 0))
+      (scale (xyz 1 1 1))
+      (rotate (xyz 0 0 0))
+    )
   )
   (module MountingHole:MountingHole_3mm (layer B.Cu)
@@
     )
     (pad 5 thru_hole circle (at 20.32 0 180) (size 3 3) (drill 1.52) (layers *.Cu *.Mask)
-      (net 5 "Net-(C4-Pad1)"))
+      (net 28 "Net-(D5-Pad1)"))
     (pad 4 thru_hole circle (at 15.24 0 180) (size 3 3) (drill 1.52) (layers *.Cu *.Mask)
-      (net 5 "Net-(C4-Pad1)"))
+      (net 28 "Net-(D5-Pad1)"))
     (pad 1 thru_hole rect (at 0 0 180) (size 3 3) (drill 1.52) (layers *.Cu *.Mask)
-      (net 5 "Net-(C4-Pad1)"))
+      (net 28 "Net-(D5-Pad1)"))
     (pad 3 thru_hole circle (at 10.16 0 180) (size 3 3) (drill 1.52) (layers *.Cu *.Mask)
-      (net 5 "Net-(C4-Pad1)"))
+      (net 28 "Net-(D5-Pad1)"))
     (pad 2 thru_hole circle (at 5.08 0 180) (size 3 3) (drill 1.52) (layers *.Cu *.Mask)
-      (net 5 "Net-(C4-Pad1)"))
+      (net 28 "Net-(D5-Pad1)"))
     (model ${KISYS3DMOD}/TerminalBlock.3dshapes/TerminalBlock_bornier-5_P5.08mm.wrl
       (offset (xyz 10.15999984741211 0 0))
@@
   (segment (start 178.91 62.74) (end 179.35 62.3) (width 0.4) (layer F.Cu) (net 4))
   (segment (start 178.91 68.5) (end 178.91 62.74) (width 0.4) (layer F.Cu) (net 4))
-  (segment (start 175.38 41.91) (end 169.47 36) (width 1) (layer F.Cu) (net 5))
-  (segment (start 169.47 36) (end 153.63 36) (width 1) (layer F.Cu) (net 5))
-  (segment (start 149.86 32.23) (end 149.86 30.48) (width 1) (layer F.Cu) (net 5))
-  (segment (start 153.63 36) (end 149.86 32.23) (width 1) (layer F.Cu) (net 5))
-  (segment (start 176.53 41.91) (end 175.38 41.91) (width 1) (layer F.Cu) (net 5))
-  (segment (start 148.11 30.48) (end 129.54 30.48) (width 1) (layer F.Cu) (net 5))
-  (segment (start 149.86 30.48) (end 148.11 30.48) (width 1) (layer F.Cu) (net 5))
+  (segment (start 148.11 30.48) (end 129.54 30.48) (width 1) (layer F.Cu) (net 28))
+  (segment (start 149.86 30.48) (end 148.11 30.48) (width 1) (layer F.Cu) (net 28))
   (segment (start 176.53 48.73) (end 179.3 51.5) (width 1) (layer F.Cu) (net 5))
   (segment (start 176.53 41.91) (end 176.53 48.73) (width 1) (layer F.Cu) (net 5))
   (segment (start 179.3 57.65) (end 179.35 57.7) (width 1) (layer F.Cu) (net 5))
   (segment (start 179.3 51.5) (end 179.3 57.65) (width 1) (layer F.Cu) (net 5))
+  (segment (start 172.8375 38.2175) (end 176.53 41.91) (width 1) (layer F.Cu) (net 5))
+  (segment (start 172.8375 37.25) (end 172.8375 38.2175) (width 1) (layer F.Cu) (net 5))
   (segment (start 167.95 54.935) (end 167.885 55) (width 0.3) (layer F.Cu) (net 6))
   (segment (start 167.95 49) (end 167.95 54.935) (width 0.3) (layer F.Cu) (net 6))
@@
   (segment (start 120.4 80.5) (end 119.75 79.85) (width 0.3) (layer F.Cu) (net 27))
   (segment (start 120.975 80.5) (end 120.4 80.5) (width 0.3) (layer F.Cu) (net 27))
+  (segment (start 154.83 37.25) (end 167.4 37.25) (width 1) (layer F.Cu) (net 28))
+  (segment (start 167.4 37.25) (end 168.1625 37.25) (width 1) (layer F.Cu) (net 28))
+  (segment (start 149.86 32.28) (end 154.83 37.25) (width 1) (layer F.Cu) (net 28))
+  (segment (start 149.86 30.48) (end 149.86 32.28) (width 1) (layer F.Cu) (net 28))
   (zone (net 4) (net_name VCC) (layer F.Cu) (hatch edge 0.508)
     (connect_pads (clearance 0.508))
